File: projectGATE/projectGATE.kicad_pcb (KiCad board)
At the start: 2 copper layers, 130 x 70 mm, 21 parts, among them J1 TB009-508-02BE, J2 TB009-508-03BE, J3 TB009-508-03BE, K1 8-1393792-5, K2 8-1393792-5, Q2 TIP41, Q3 TIP41, U1 ESP32-DEVKITC, U2 PC817, U3 PC817

Commit message: fix
Parts:
- PS1: value VOF-S12B-5 -> HLK-PM01; footprint VOF-S12B-5:CONV_VOF-S12B-5 -> HLK-PM01:CONV_HLK-PM01
- moved J1 3.55 mm to (99.0, 87.0)
- moved PS1 3.39 mm to (101.0, 114.0)
Connections:
- PS1 pad 3: GND -> 5V
- PS1 pad 4: 5V -> GND
Routing:
- net 5V: track 320.5 -> 325.6 mm
- net GND: track 241.5 -> 245.6 mm
- net Net-(PS1-AC1): track 18.5 -> 15.9 mm
- net Net-(PS1-AC2): track 12.3 -> 14.2 mm
